File: Lora58thsStubShunt.kicad_pcb (KiCad board)
At the start: 2 copper layers, 35.5 x 18.5 mm, 9 parts, among them J1 Conn_Coaxial, J2 Conn_01x01_Pin, J3 Conn_01x01_Pin, J4 Conn_01x01_Pin

Commit message: Release Candidate
Parts:
- removed NT1: NetTie_2, Jumper:SolderJumper-2_P1.3mm_Open_RoundedPad1.0x1.5mm
- moved C1 2.53 mm to (91.0, 82.5)
- moved C2 2.53 mm to (91.0, 83.5)
Routing:
- net Net-(J1-In): track 91.6 -> 13.4 mm
- net Net-(J2-Pin_1): track 6.87 -> 4.65 mm
- net GND: track 5.31 -> 4.60 mm
Other:
- board size 35.5 x 18.5 mm -> 35.5 x 12.3 mm
- board text removed: "79.5mm"
